File: PCB/mounting_holes.kicad_sch (KiCad schematic)
At the start: 13 parts

Commit message: First commit, removed unnecessary files, ChatGPT'd the readme, added production and Kicad files for Left&Right sides as well as the Plate.
Parts:
- added H12, H13, H14, H15, H16, H17: Black_Screws, cipulot_parts:HOLE_M2_RF, symbol Mechanical:MountingHole
